Commit message: new nav2 params, camera added

File: models/rover/rover.urdf (robot description, URDF)
Before this commit: robot seamk_rover, 5 links, 4 joints
Links:
- added link camera_link
Joints:
- added joint camera_joint: type fixed, parent base_link, child camera_link, origin xyz=0.4 0 0.1 rpy=0 0 0
